File: openSX70-bench/openSX70-bench-new.brd (EAGLE design)
At the start: 99.3 x 100.2 mm, 42 parts

Commit message: Working on the bench and on the charger
Parts:
- removed JP1: (no value), pinhead:1X07
- removed SONAR: (no value), pinhead:1X08
- added FLEXCABLE: (no value), pinhead:1X07
- added H5, H6: MOUNT-HOLE2.8, holes:2,8
- added SONAR_FLASHFLEX: (no value), pinhead:1X08
- moved S2 83.3 mm to (55.1, 9.20), turned to 0 degrees
- moved SOL2 83.1 mm to (37.4, 8.69)
- moved VCC 55.9 mm to (29.6, 92.1)
- moved FLASH 20.5 mm to (91.0, 9.09)
- moved ICSP 16.5 mm to (92.0, 23.2)
- moved S1 8.02 mm to (45.6, 9.14), turned to 0 degrees
- moved GNDS 6.53 mm to (10.1, 92.6), turned to 0 degrees
- moved S1-COMMON 2.81 mm to (9.95, 57.1), turned to 90 degrees
- moved S1-T 2.80 mm to (5.44, 57.0)
- moved S1-F 2.78 mm to (7.76, 57.8)
- moved SOL1 2.30 mm to (27.1, 8.60)
- moved SOL2+ 0.34 mm to (15.1, 57.1)
- moved RST 0.28 mm to (66.9, 42.0)
- moved SOL2+1 0.20 mm to (12.2, 57.3)
Connections:
- removed net N$11: SONAR.8
- removed net N$19: SONAR.2, U$2.VCC
- removed net N$27: SOL1+.1, SOL1.2
- removed net N$3: JP1.5, U$1.VCC
- removed net N$5: JP1.3, U$1.GND
- new net 6V-SOL1: SOL1+.1, SOL1.2, VCC.4
- net 6V-I: no longer VCC.4
- net 6V-S: now also SONAR_FLASHFLEX.2, U$2.VCC
- net GND-C: now also FLEXCABLE.3, U$1.GND
- net GND-I: now also GND-2.1
- net GND-S: now also SONAR_FLASHFLEX.8; no longer GND-2.1
- net N$1: now also FLEXCABLE.7; no longer JP1.7
- net N$13: now also SONAR_FLASHFLEX.7; no longer SONAR.7
- net N$14: now also SONAR_FLASHFLEX.6; no longer SONAR.6
- net N$15: now also SONAR_FLASHFLEX.5; no longer SONAR.5
- net N$16: now also SONAR_FLASHFLEX.1; no longer SONAR.1
- net N$17: now also SONAR_FLASHFLEX.3; no longer SONAR.3
- net N$18: now also SONAR_FLASHFLEX.4; no longer SONAR.4
- net N$2: now also FLEXCABLE.6; no longer JP1.6
- net N$4: now also FLEXCABLE.4; no longer JP1.4
- net N$6: now also FLEXCABLE.2; no longer JP1.2
- net N$7: now also FLEXCABLE.1; no longer JP1.1
- net VCC-C: now also FLEXCABLE.5, U$1.VCC

Commit message: Working on the bench
Parts:
- added FLASH1, SOL3: (no value), pinhead:1X04
- added FLEXCABLE1: (no value), pinhead:1X07
- added ICSP1: (no value), pinhead:2X03
- added S3, SOL4: (no value), pinhead:1X02
- added S4: (no value), pinhead:1X03
- added SONAR_FLASHFLEX1: (no value), pinhead:1X08
- moved SOL1 2.95 mm to (27.9, 11.4)
- moved VCC 2.89 mm to (27.2, 90.5)
- moved FLEXCABLE 2.80 mm to (11.8, 11.4)
- moved SOL2 2.77 mm to (37.7, 11.4)
- moved S1 2.38 mm to (46.2, 11.4)
- moved FLASH 2.35 mm to (91.0, 11.4)
- moved SONAR_FLASHFLEX 2.29 mm to (69.6, 11.4)
- moved S2 2.27 mm to (54.8, 11.4)
- moved GNDS 2.16 mm to (10.1, 90.5)
- moved XTRAS 1.99 mm to (60.4, 90.5)
- moved ICSP 0.34 mm to (92.3, 23.2)
- moved BA 0.18 mm to (23.3, 39.8)
- moved BC 0.14 mm to (21.4, 39.9)
Connections:
- net 6V-F: now also FLASH1.3
- net 6V-I: now also ICSP1.2
- net 6V-S: now also SONAR_FLASHFLEX1.2
- net 6V-SOL1: now also SOL3.2
- net GND-C: now also FLEXCABLE1.3
- net GND-F: now also FLASH1.1
- net GND-I: now also ICSP1.6
- net GND-S: now also SONAR_FLASHFLEX1.8
- net N$1: now also FLEXCABLE1.7
- net N$10: now also ICSP1.5
- net N$12: now also ICSP1.4
- net N$13: now also SONAR_FLASHFLEX1.7
- net N$14: now also SONAR_FLASHFLEX1.6
- net N$15: now also SONAR_FLASHFLEX1.5
- net N$16: now also SONAR_FLASHFLEX1.1
- net N$17: now also SONAR_FLASHFLEX1.3
- net N$18: now also SONAR_FLASHFLEX1.4
- net N$2: now also FLEXCABLE1.6
- net N$21: now also S4.3
- net N$22: now also S4.2
- net N$23: now also FLASH1.2
- net N$24: now also S4.1
- net N$25: now also FLASH1.4
- net N$26: now also SOL3.1
- net N$28: now also SOL3.3
- net N$29: now also SOL3.4
- net N$34: now also SOL4.1
- net N$35: now also SOL4.2
- net N$38: now also S3.1
- net N$39: now also S3.2
- net N$4: now also FLEXCABLE1.4
- net N$6: now also FLEXCABLE1.2
- net N$7: now also FLEXCABLE1.1
- net N$8: now also ICSP1.1
- net N$9: now also ICSP1.3
- net VCC-C: now also FLEXCABLE1.5
Other:
- board text added: "GND"
- board text added: "MOTOR"
- board text added: "S1C"
- board text added: "S1F"
- board text added: "S1T"
- board text added: "S3"
- board text added: "S5"
- board text added: "S8"
- board text added: "S9"
- board text added: "SOL1+"
- board text added: "SOL1-"
- board text added: "SOL1A"
- board text added: "SOL1B"
- board text added: "SOL2+"
- board text added: "VCC"

Commit message: minor progress on the bench
Parts:
- removed XTRAS: (no value), pinhead:1X03
- moved SONAR_FLASHFLEX 0.42 mm to (70.1, 11.4), turned to 180 degrees
- flipped SONAR_FLASHFLEX1 to the bottom
Other:
- board text added: "F+"
- board text added: "F-"
- board text added: "FF"
- board text added: "FT"
- board text added: "GTD"
- board text added: "S2"
- board text added: "openSX70 universal bench tester v.2.0"

Commit message: the bench v.2
Parts:
- added XA1, XA2, XA3, XA4: 5-534237-8, Common-Parts-Library-Eagle:TE_5-534237-8
- moved SONAR_FLASHFLEX 0.27 mm to (69.8, 11.4)
Connections:
- new net N$11: XA4.3, XA4.4
- new net N$19: XA4.5, XA4.6
- new net N$27: XA4.10, XA4.9
- new net N$3: XA1.1, XA1.10, XA1.2, XA1.3, XA1.4, XA1.5, XA1.6, XA1.7, XA1.8, XA1.9
- new net N$30: XA2.1, XA2.2, XA2.3, XA2.4, XA2.5
- new net N$31: XA2.10, XA2.6, XA2.7, XA2.8, XA2.9
- new net N$5: XA4.1, XA4.2
- net GND-I: no longer GND-2.1
- net GND-S: now also GND-2.1, U$2.GND
- net N$20: now also XA4.7, XA4.8; no longer U$2.GND
Routing:
- net GND-S: track 0.00 -> 249.4 mm, vias 0 -> 3
- net GND-I: track 0.00 -> 227.0 mm, vias 0 -> 3
- net GND-F: track 0.00 -> 156.4 mm, vias 0 -> 3
- net 6V-S: track 0.00 -> 135.1 mm
- net N$13: track 0.00 -> 127.3 mm, vias 0 -> 1
- net N$14: track 0.00 -> 123.4 mm, vias 0 -> 3
- net 6V-F: track 0.00 -> 122.6 mm, vias 0 -> 1
- net N$9: track 0.00 -> 106.1 mm, vias 0 -> 2
- net N$10: track 0.00 -> 105.0 mm
- net N$8: track 0.00 -> 104.3 mm
- net N$12: track 0.00 -> 102.2 mm, vias 0 -> 2
- net 6V-SOL1: track 0.00 -> 95.1 mm
- net VCC-C: track 0.00 -> 94.2 mm, vias 0 -> 2
- net GND-C: track 0.00 -> 93.0 mm, vias 0 -> 2
- net 6V-I: track 0.00 -> 88.0 mm, vias 0 -> 1
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Other:
- board text added: "FLASH"
- board text added: "FLEX"
- board text added: "ICSP"
- board text added: "MISO"
- board text added: "MOSI"
- board text added: "RST"
- board text added: "SCK"
- board text added: "SOL1"
- board text added: "SONAR"
