File: openSX70-bench/openSX70-bench-new.sch (EAGLE design)
At the start: 42 parts

Commit message: Working on the bench and on the charger
Parts:
- renumbered JP1 to FLEXCABLE, SONAR to SONAR_FLASHFLEX
Connections:
- removed net N$11: SONAR_FLASHFLEX.8
- removed net N$19: SONAR_FLASHFLEX.2, U$2.VCC
- removed net N$27: SOL1+.KL, SOL1.2
- removed net N$3: FLEXCABLE.5, U$1.6V
- removed net N$5: FLEXCABLE.3, U$1.GND
- new net 6V-SOL1: SOL1+.KL, SOL1.2, VCC.4
- net 6V-I: no longer VCC.4
- net 6V-S: now also SONAR_FLASHFLEX.2, U$2.VCC
- net GND-C: now also FLEXCABLE.3, U$1.GND
- net GND-I: now also GND-2.KL
- net GND-S: now also SONAR_FLASHFLEX.8; no longer GND-2.KL
- net VCC-C: now also FLEXCABLE.5, U$1.6V

Commit message: Working on the bench
Parts:
- added FLASH1, SOL3: (no value), pinhead:PINHD-1X4
- added FLEXCABLE1: (no value), pinhead:PINHD-1X7
- added ICSP1: (no value), pinhead:PINHD-2X3
- added S3, SOL4: (no value), pinhead:PINHD-1X2
- added S4: (no value), pinhead:PINHD-1X3
- added SONAR_FLASHFLEX1: (no value), pinhead:PINHD-1X8
Connections:
- net 6V-F: now also FLASH1.3
- net 6V-I: now also ICSP1.2
- net 6V-S: now also SONAR_FLASHFLEX1.2
- net 6V-SOL1: now also SOL3.2
- net GND-C: now also FLEXCABLE1.3
- net GND-F: now also FLASH1.1
- net GND-I: now also ICSP1.6
- net GND-S: now also SONAR_FLASHFLEX1.8
- net N$1: now also FLEXCABLE1.7
- net N$10: now also ICSP1.5
- net N$12: now also ICSP1.4
- net N$13: now also SONAR_FLASHFLEX1.7
- net N$14: now also SONAR_FLASHFLEX1.6
- net N$15: now also SONAR_FLASHFLEX1.5
- net N$16: now also SONAR_FLASHFLEX1.1
- net N$17: now also SONAR_FLASHFLEX1.3
- net N$18: now also SONAR_FLASHFLEX1.4
- net N$2: now also FLEXCABLE1.6
- net N$21: now also S4.3
- net N$22: now also S4.2
- net N$23: now also FLASH1.2
- net N$24: now also S4.1
- net N$25: now also FLASH1.4
- net N$26: now also SOL3.1
- net N$28: now also SOL3.3
- net N$29: now also SOL3.4
- net N$34: now also SOL4.1
- net N$35: now also SOL4.2
- net N$38: now also S3.1
- net N$39: now also S3.2
- net N$4: now also FLEXCABLE1.4
- net N$6: now also FLEXCABLE1.2
- net N$7: now also FLEXCABLE1.1
- net N$8: now also ICSP1.1
- net N$9: now also ICSP1.3
- net VCC-C: now also FLEXCABLE1.5

Commit message: minor progress on the bench
Parts:
- removed XTRAS: (no value), pinhead:PINHD-1X3
Changed lines of the file:
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@@
 <part name="S2" library="pinhead" library_urn="urn:adsk.eagle:library:325" deviceset="PINHD-1X2" device="" package3d_urn="urn:adsk.eagle:package:22435/2"/>
 <part name="SONAR_FLASHFLEX" library="pinhead" library_urn="urn:adsk.eagle:library:325" deviceset="PINHD-1X8" device="" package3d_urn="urn:adsk.eagle:package:22409/2"/>
-<part name="XTRAS" library="pinhead" library_urn="urn:adsk.eagle:library:325" deviceset="PINHD-1X3" device="" package3d_urn="urn:adsk.eagle:package:22458/2"/>
 <part name="VCC" library="pinhead" library_urn="urn:adsk.eagle:library:325" deviceset="PINHD-1X4" device="" package3d_urn="urn:adsk.eagle:package:22407/2"/>
 <part name="GNDS" library="pinhead" library_urn="urn:adsk.eagle:library:325" deviceset="PINHD-1X4" device="" package3d_urn="urn:adsk.eagle:package:22407/2"/>
@@
 <attribute name="VALUE" x="52.07" y="132.08" size="1.778" layer="96"/>
 </instance>
-<instance part="XTRAS" gate="A" x="223.52" y="154.94">
-<attribute name="NAME" x="217.17" y="160.655" size="1.778" layer="95"/>
-<attribute name="VALUE" x="217.17" y="147.32" size="1.778" layer="96"/>
-</instance>
 <instance part="VCC" gate="A" x="246.38" y="81.28" rot="R180">

Commit message: the bench v.2
Parts:
- added XA1, XA2, XA3, XA4: 5-534237-8, Common-Parts-Library-Eagle:5-534237-8
Connections:
- new net N$11: XA4.3, XA4.4
- new net N$19: XA4.5, XA4.6
- new net N$27: XA4.10, XA4.9
- new net N$3: XA1.1, XA1.10, XA1.2, XA1.3, XA1.4, XA1.5, XA1.6, XA1.7, XA1.8, XA1.9
- new net N$30: XA2.1, XA2.2, XA2.3, XA2.4, XA2.5
- new net N$31: XA2.10, XA2.6, XA2.7, XA2.8, XA2.9
- new net N$5: XA4.1, XA4.2
- net GND-I: no longer GND-2.KL
- net GND-S: now also GND-2.KL, U$2.-
- net N$20: now also XA4.7, XA4.8; no longer U$2.-
Other:
- moved on the sheet: S4
Changed lines of the file:
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@@
 </variantdefs>
 <classes>
-<class number="0" name="default" width="0.6096" drill="0">
+<class number="0" name="default" width="0.3048" drill="0">
+</class>
+<class number="1" name="GND" width="0.508" drill="0">
+</class>
+<class number="2" name="VCC" width="0.508" drill="0">
 </class>
 </classes>
@@
 <part name="S4" library="pinhead" library_urn="urn:adsk.eagle:library:325" deviceset="PINHD-1X3" device="" package3d_urn="urn:adsk.eagle:package:22458/2"/>
 <part name="ICSP1" library="pinhead" library_urn="urn:adsk.eagle:library:325" deviceset="PINHD-2X3" device="" package3d_urn="urn:adsk.eagle:package:22462/2"/>
+<part name="XA1" library="Common-Parts-Library-Eagle" deviceset="5-534237-8" device=""/>
+<part name="XA2" library="Common-Parts-Library-Eagle" deviceset="5-534237-8" device=""/>
+<part name="XA3" library="Common-Parts-Library-Eagle" deviceset="5-534237-8" device=""/>
+<part name="XA4" library="Common-Parts-Library-Eagle" deviceset="5-534237-8" device=""/>
 </parts>
 <sheets>
@@
 <attribute name="VALUE" x="77.47" y="40.64" size="1.778" layer="96"/>
 </instance>
-<instance part="S4" gate="A" x="73.66" y="20.32">
-<attribute name="NAME" x="67.31" y="26.035" size="1.778" layer="95"/>
-<attribute name="VALUE" x="67.31" y="12.7" size="1.778" layer="96"/>
+<instance part="S4" gate="A" x="71.12" y="20.32">
+<attribute name="NAME" x="64.77" y="26.035" size="1.778" layer="95"/>
+<attribute name="VALUE" x="64.77" y="12.7" size="1.778" layer="96"/>
 </instance>
 <instance part="ICSP1" gate="A" x="167.64" y="15.24">
 <attribute name="NAME" x="161.29" y="20.955" size="1.778" layer="95"/>
 <attribute name="VALUE" x="161.29" y="7.62" size="1.778" layer="96"/>
+</instance>
+<instance part="XA1" gate="G$1" x="172.72" y="170.18" rot="R90">
+<attribute name="NAME" x="158.115" y="166.37" size="1.778" layer="95" rot="R90"/>
+<attribute name="VALUE" x="189.23" y="166.37" size="1.778" layer="96" rot="R90"/>
+</instance>
+<instance part="XA2" gate="G$1" x="218.44" y="160.02" rot="R90">
+<attribute name="NAME" x="203.835" y="156.21" size="1.778" layer="95" rot="R90"/>
+<attribute name="VALUE" x="234.95" y="156.21" size="1.778" layer="96" rot="R90"/>
+</instance>
+<instance part="XA3" gate="G$1" x="220.98" y="139.7" rot="R90">
+<attribute name="NAME" x="206.375" y="135.89" size="1.778" layer="95" rot="R90"/>
+<attribute name="VALUE" x="237.49" y="135.89" size="1.778" layer="96" rot="R90"/>
+</instance>
+<instance part="XA4" gate="G$1" x="182.88" y="144.78" rot="R90">
+<attribute name="NAME" x="168.275" y="140.97" size="1.778" layer="95" rot="R90"/>
+<attribute name="VALUE" x="199.39" y="140.97" size="1.778" layer="96" rot="R90"/>
 </instance>
 </instances>
@@
 <label x="269.24" y="68.58" size="1.778" layer="95"/>
 </segment>
-<segment>
-<pinref part="GND-2" gate="G$1" pin="KL"/>
-<wire x1="0" y1="129.54" x2="5.08" y2="129.54" width="0.1524" layer="91"/>
-<label x="5.08" y="132.08" size="1.778" layer="95"/>
-</segment>
 </net>
 <net name="6V-S" class="0">
@@
 <junction x="55.88" y="137.16"/>
 </segment>
+<segment>
+<pinref part="GND-2" gate="G$1" pin="KL"/>
+<wire x1="0" y1="129.54" x2="5.08" y2="129.54" width="0.1524" layer="91"/>
+<label x="5.08" y="132.08" size="1.778" layer="95"/>
+</segment>
+<segment>
+<pinref part="U$2" gate="G$1" pin="-"/>
+<wire x1="30.48" y1="129.54" x2="48.26" y2="129.54" width="0.1524" layer="91"/>
+<label x="40.64" y="127" size="1.778" layer="95" rot="R180"/>
+</segment>
 </net>
 <net name="N$13" class="0">
@@
 </segment>
 </net>
-<net name="N$20" class="0">
-<segment>
-<pinref part="U$2" gate="G$1" pin="-"/>
-<wire x1="30.48" y1="129.54" x2="48.26" y2="129.54" width="0.1524" layer="91"/>
-</segment>
-</net>
 <net name="N$1" class="0">
 <segment>
@@
 <pinref part="S1" gate="A" pin="3"/>
 <pinref part="S4" gate="A" pin="3"/>
-<wire x1="71.12" y1="17.78" x2="58.42" y2="17.78" width="0.1524" layer="91"/>
+<wire x1="68.58" y1="17.78" x2="58.42" y2="17.78" width="0.1524" layer="91"/>
 <junction x="58.42" y="17.78"/>
 </segment>
@@
 <pinref part="S1" gate="A" pin="2"/>
 <pinref part="S4" gate="A" pin="2"/>
-<wire x1="58.42" y1="20.32" x2="71.12" y2="20.32" width="0.1524" layer="91"/>
+<wire x1="58.42" y1="20.32" x2="68.58" y2="20.32" width="0.1524" layer="91"/>
 <junction x="58.42" y="20.32"/>
 </segment>
@@
 <pinref part="S1" gate="A" pin="1"/>
 <pinref part="S4" gate="A" pin="1"/>
-<wire x1="58.42" y1="22.86" x2="71.12" y2="22.86" width="0.1524" layer="91"/>
+<wire x1="58.42" y1="22.86" x2="68.58" y2="22.86" width="0.1524" layer="91"/>
 <junction x="58.42" y="22.86"/>
 </segment>
 </net>
+<net name="N$3" class="0">
+<segment>
+<pinref part="XA1" gate="G$1" pin="1"/>
+<pinref part="XA1" gate="G$1" pin="2"/>
+<wire x1="161.29" y1="161.29" x2="163.83" y2="161.29" width="0.1524" layer="91"/>
+<pinref part="XA1" gate="G$1" pin="3"/>
+<wire x1="163.83" y1="161.29" x2="166.37" y2="161.29" width="0.1524" layer="91"/>
+<junction x="163.83" y="161.29"/>
+<pinref part="XA1" gate="G$1" pin="4"/>
+<wire x1="166.37" y1="161.29" x2="168.91" y2="161.29" width="0.1524" layer="91"/>
+<junction x="166.37" y="161.29"/>
+<pinref part="XA1" gate="G$1" pin="5"/>
+<wire x1="168.91" y1="161.29" x2="171.45" y2="161.29" width="0.1524" layer="91"/>
+<junction x="168.91" y="161.29"/>
+<pinref part="XA1" gate="G$1" pin="6"/>
+<wire x1="171.45" y1="161.29" x2="173.99" y2="161.29" width="0.1524" layer="91"/>
+<junction x="171.45" y="161.29"/>
+<pinref part="XA1" gate="G$1" pin="7"/>
+<wire x1="173.99" y1="161.29" x2="176.53" y2="161.29" width="0.1524" layer="91"/>
+<junction x="173.99" y="161.29"/>
+<pinref part="XA1" gate="G$1" pin="8"/>
+<wire x1="176.53" y1="161.29" x2="179.07" y2="161.29" width="0.1524" layer="91"/>
+<junction x="176.53" y="161.29"/>
+<pinref part="XA1" gate="G$1" pin="9"/>
+<wire x1="179.07" y1="161.29" x2="181.61" y2="161.29" width="0.1524" layer="91"/>
+<junction x="179.07" y="161.29"/>
+<pinref part="XA1" gate="G$1" pin="10"/>
+<wire x1="181.61" y1="161.29" x2="184.15" y2="161.29" width="0.1524" layer="91"/>
+<junction x="181.61" y="161.29"/>
+</segment>
+</net>
+<net name="N$5" class="0">
+<segment>
+<pinref part="XA4" gate="G$1" pin="1"/>
+<pinref part="XA4" gate="G$1" pin="2"/>
+<wire x1="171.45" y1="135.89" x2="173.99" y2="135.89" width="0.1524" layer="91"/>
+</segment>
+</net>
+<net name="N$11" class="0">
+<segment>
+<pinref part="XA4" gate="G$1" pin="3"/>
+<pinref part="XA4" gate="G$1" pin="4"/>
+<wire x1="176.53" y1="135.89" x2="179.07" y2="135.89" width="0.1524" layer="91"/>
+</segment>
+</net>
+<net name="N$19" class="0">
+<segment>
+<pinref part="XA4" gate="G$1" pin="6"/>
+<wire x1="182.88" y1="137.16" x2="184.15" y2="137.16" width="0.1524" layer="91"/>
+<wire x1="184.15" y1="137.16" x2="184.15" y2="135.89" width="0.1524" layer="91"/>
+<pinref part="XA4" gate="G$1" pin="5"/>
+<wire x1="181.61" y1="135.89" x2="184.15" y2="135.89" width="0.1524" layer="91"/>
+<junction x="184.15" y="135.89"/>
+</segment>
+</net>
+<net name="N$20" class="0">
+<segment>
+<pinref part="XA4" gate="G$1" pin="7"/>
+<pinref part="XA4" gate="G$1" pin="8"/>
+<wire x1="186.69" y1="135.89" x2="189.23" y2="135.89" width="0.1524" layer="91"/>
+</segment>
+</net>
+<net name="N$27" class="0">
+<segment>
+<pinref part="XA4" gate="G$1" pin="9"/>
+<pinref part="XA4" gate="G$1" pin="10"/>
+<wire x1="191.77" y1="135.89" x2="194.31" y2="135.89" width="0.1524" layer="91"/>
+</segment>
+</net>
+<net name="N$30" class="0">
+<segment>
+<pinref part="XA2" gate="G$1" pin="1"/>
+<pinref part="XA2" gate="G$1" pin="2"/>
+<wire x1="207.01" y1="151.13" x2="209.55" y2="151.13" width="0.1524" layer="91"/>
+<pinref part="XA2" gate="G$1" pin="3"/>
+<wire x1="209.55" y1="151.13" x2="212.09" y2="151.13" width="0.1524" layer="91"/>
+<junction x="209.55" y="151.13"/>
+<pinref part="XA2" gate="G$1" pin="4"/>
+<wire x1="212.09" y1="151.13" x2="214.63" y2="151.13" width="0.1524" layer="91"/>
+<junction x="212.09" y="151.13"/>
+<pinref part="XA2" gate="G$1" pin="5"/>
+<wire x1="214.63" y1="151.13" x2="217.17" y2="151.13" width="0.1524" layer="91"/>
+<junction x="214.63" y="151.13"/>
+</segment>
+</net>
+<net name="N$31" class="0">
+<segment>
+<pinref part="XA2" gate="G$1" pin="6"/>
+<pinref part="XA2" gate="G$1" pin="7"/>
+<wire x1="219.71" y1="151.13" x2="222.25" y2="151.13" width="0.1524" layer="91"/>
+<pinref part="XA2" gate="G$1" pin="8"/>
+<wire x1="222.25" y1="151.13" x2="224.79" y2="151.13" width="0.1524" layer="91"/>
+<junction x="222.25" y="151.13"/>
+<pinref part="XA2" gate="G$1" pin="9"/>
+<wire x1="224.79" y1="151.13" x2="227.33" y2="151.13" width="0.1524" layer="91"/>
+<junction x="224.79" y="151.13"/>
+<pinref part="XA2" gate="G$1" pin="10"/>
+<wire x1="227.33" y1="151.13" x2="229.87" y2="151.13" width="0.1524" layer="91"/>
+<junction x="227.33" y="151.13"/>
+</segment>
+</net>
