File: openSX70-bench/openSX70-bench-new-v2-1.sch (EAGLE design)
At the start: 53 parts

Commit message: bench final-production
Parts:
- U$2: device openSX70:SX70-SONAR-FLASHFLEX-HOLES -> _openSX70:SX70-SONAR-FLASHFLEX-HOLES
Changed lines of the file:
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@@
 <part name="GNDS" library="pinhead" library_urn="urn:adsk.eagle:library:325" deviceset="PINHD-1X4" device="" package3d_urn="urn:adsk.eagle:package:22407/2"/>
 <part name="U$1" library="openSX70" deviceset="SX70-7-PAD-HOLES-PROPER" device=""/>
-<part name="U$2" library="openSX70" deviceset="SX70-SONAR-FLASHFLEX-HOLES" device=""/>
+<part name="U$2" library="_openSX70" deviceset="SX70-SONAR-FLASHFLEX-HOLES" device=""/>
 <part name="FLEXCABLE" library="pinhead" library_urn="urn:adsk.eagle:library:325" deviceset="PINHD-1X7" device="" package3d_urn="urn:adsk.eagle:package:22477/2"/>
 <part name="H1" library="holes" library_urn="urn:adsk.eagle:library:237" deviceset="MOUNT-HOLE" device="2.8" package3d_urn="urn:adsk.eagle:package:14271/1"/>
@@
 </instance>
 <instance part="U$1" gate="G$1" x="40.64" y="109.22" rot="MR270"/>
-<instance part="U$2" gate="G$1" x="66.04" y="142.24"/>
+<instance part="U$2" gate="G$1" x="17.78" y="147.32"/>
 <instance part="FLEXCABLE" gate="A" x="40.64" y="78.74" rot="R270">
 <attribute name="NAME" x="51.435" y="85.09" size="1.778" layer="95" rot="R270"/>
@@
 </drawing>
 <compatibility>
-<note version="6.3" minversion="6.2.2" severity="warning">
-Since Version 6.2.2 text objects can contain more than one line,
-which will not be processed correctly with this version.
-</note>
 <note version="8.2" severity="warning">
 Since Version 8.2, EAGLE supports online libraries. The ids
