File: openSX70-bench/openSX70-bench-new-v2-3.brd (EAGLE design)
At the start: 99.3 x 100.2 mm, 59 parts

Commit message: New version
Parts:
- added JP1, JP2: (no value), pinhead:1X01
Connections:
- new net N$32: JP1.1, JP2.1, S2B.1
- net N$13: no longer S2B.1
Routing:
- net N$32: track 0.00 -> 75.1 mm, vias 0 -> 1
- net N$13: track 127.4 -> 103.7 mm
Other:
- board text added: "S2+"
- board text added: "S2-"
- board text added: "S2B"
- board text added: "S2B+"
- board text added: "SOL2-"
Changed lines of the file:
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@@
 <text x="17.91" y="6.5" size="1.778" layer="25" font="vector" rot="R90">S9</text>
 <text x="20.5" y="6.45" size="1.778" layer="25" font="vector" rot="R90">S8</text>
-<text x="25.4" y="2.54" size="1.778" layer="25" font="vector" rot="R90">SOL1+</text>
-<text x="27.94" y="2.54" size="1.778" layer="25" font="vector" rot="R90">SOL1-</text>
+<text x="25.4" y="2.54" size="1.778" layer="25" font="vector" rot="R90">SOL1-</text>
+<text x="27.94" y="2.54" size="1.778" layer="25" font="vector" rot="R90">SOL1+</text>
 <text x="30.48" y="2.54" size="1.778" layer="25" font="vector" rot="R90">SOL1B</text>
 <text x="33.02" y="2.54" size="1.778" layer="25" font="vector" rot="R90">SOL1A</text>
 <text x="38.1" y="2.54" size="1.778" layer="25" font="vector" rot="R90">SOL2+</text>
-<text x="40.64" y="2.54" size="1.778" layer="25" font="vector" rot="R90">SOL2+</text>
+<text x="40.64" y="2.54" size="1.778" layer="25" font="vector" rot="R90">SOL2-</text>
 <text x="44.58" y="5.35" size="1.778" layer="25" font="vector" rot="R90">S1T</text>
 <text x="47.39" y="5.43" size="1.778" layer="25" font="vector" rot="R90">S1C</text>
@@
 <text x="32.84" y="58.87" size="1.778" layer="25" font="vector" rot="R234.4">GTD</text>
 <rectangle x1="2.54" y1="17.78" x2="83.82" y2="33.02" layer="22"/>
+<text x="56.9" y="5.15" size="1.778" layer="25" font="vector" rot="R90">S2-</text>
+<text x="-26.84" y="105.53" size="1.778" layer="25" font="vector" rot="R270">S2B</text>
+<wire x1="76.032" y1="77.698" x2="76.032" y2="72.11" width="0.1524" layer="21"/>
+<wire x1="76.032" y1="72.11" x2="81.112" y2="72.11" width="0.1524" layer="21"/>
+<wire x1="81.112" y1="72.11" x2="81.112" y2="77.698" width="0.1524" layer="21"/>
+<wire x1="81.112" y1="77.698" x2="76.032" y2="77.698" width="0.1524" layer="21"/>
+<wire x1="76.54" y1="77.19" x2="80.604" y2="77.19" width="0.1524" layer="21"/>
+<wire x1="80.604" y1="77.19" x2="80.604" y2="73.507" width="0.1524" layer="21"/>
+<wire x1="80.604" y1="73.507" x2="76.54" y2="73.507" width="0.1524" layer="21"/>
+<wire x1="76.54" y1="73.507" x2="76.54" y2="77.19" width="0.1524" layer="21"/>
+<rectangle x1="76.59" y1="73.505" x2="80.545" y2="77.19" layer="21"/>
+<text x="54.37" y="5.16" size="1.778" layer="25" font="vector" rot="R90">S2+</text>
+<text x="83.88" y="3.5" size="1.778" layer="25" font="vector" rot="R90">S2B+</text>
 </plain>
 <attributes>
@@
 <element name="H9" library="holes" library_urn="urn:adsk.eagle:library:237" package="2,8" package3d_urn="urn:adsk.eagle:package:14271/1" value="MOUNT-HOLE2.8" x="4" y="4" smashed="yes"/>
 <element name="H10" library="holes" library_urn="urn:adsk.eagle:library:237" package="2,8" package3d_urn="urn:adsk.eagle:package:14271/1" value="MOUNT-HOLE2.8" x="4" y="96" smashed="yes"/>
+<element name="JP1" library="pinhead" library_urn="urn:adsk.eagle:library:325" package="1X01" package3d_urn="urn:adsk.eagle:package:22485/2" value="" x="83.08" y="15.48" smashed="yes">
+<attribute name="VALUE" x="81.81" y="12.305" size="1.27" layer="27"/>
+</element>
+<element name="JP2" library="pinhead" library_urn="urn:adsk.eagle:library:325" package="1X01" package3d_urn="urn:adsk.eagle:package:22485/2" value="" x="83.13" y="11.29" smashed="yes">
+<attribute name="VALUE" x="81.86" y="8.115" size="1.27" layer="27"/>
+</element>
 </elements>
 <signals>
@@
 <wire x1="56" y1="15.5" x2="32.5" y2="39" width="0.3048" layer="1"/>
 <wire x1="28.5" y1="62.5" x2="28.34" y2="62.58" width="0.3048" layer="16"/>
+<via x="32.5" y="39" extent="1-16" drill="0.35"/>
 <wire x1="56" y1="15.5" x2="56.112" y2="15.56" width="0.3048" layer="1"/>
-<via x="32.5" y="39" extent="1-16" drill="0.35"/>
 </signal>
 <signal name="GND-F">
@@
 <contactref element="SONAR_FLASHFLEX" pad="7"/>
 <contactref element="U$2" pad="S2"/>
-<contactref element="S2B" pad="1"/>
 <contactref element="SONAR_FLASHFLEX1" pad="7"/>
 <wire x1="23.076225" y1="48.0143" x2="22.3616" y2="48.728925" width="0.3048" layer="1"/>
@@
 <wire x1="63.5" y1="17.78" x2="63.39" y2="15.56" width="0.3048" layer="1"/>
 <wire x1="63.39" y1="15.56" x2="63.44" y2="11.44" width="0.3048" layer="1"/>
-<wire x1="82.5" y1="55" x2="88" y2="60.5" width="0.3048" layer="1"/>
-<wire x1="82.5" y1="39.5" x2="82.5" y2="55" width="0.3048" layer="1"/>
 <wire x1="64" y1="21" x2="82.5" y2="39.5" width="0.3048" layer="16"/>
 <wire x1="64" y1="16" x2="64" y2="21" width="0.3048" layer="16"/>
 <wire x1="63.5" y1="16" x2="64" y2="16" width="0.3048" layer="16"/>
-<wire x1="88" y1="60.5" x2="88.4" y2="60.6" width="0.3048" layer="1"/>
 <wire x1="63.5" y1="16" x2="63.39" y2="15.56" width="0.3048" layer="16"/>
 <via x="82.5" y="39.5" extent="1-16" drill="0.35"/>
@@
 <wire x1="67.31" y1="83.82" x2="69.85" y2="83.82" width="0.3048" layer="1"/>
 </signal>
+<signal name="N$32">
+<contactref element="S2B" pad="1"/>
+<contactref element="JP1" pad="1"/>
+<contactref element="JP2" pad="1"/>
+<wire x1="83.08" y1="15.48" x2="83.08" y2="11.34" width="0.3048" layer="1"/>
+<wire x1="83.08" y1="11.34" x2="83.13" y2="11.29" width="0.3048" layer="1"/>
+<wire x1="83.13" y1="11.29" x2="85.4" y2="13.56" width="0.3048" layer="16"/>
+<wire x1="85.4" y1="13.56" x2="97.42" y2="13.56" width="0.3048" layer="16"/>
+<wire x1="97.42" y1="13.56" x2="97.42" y2="31.9" width="0.3048" layer="16"/>
+<wire x1="90.08" y1="39.24" x2="90.08" y2="40.73" width="0.3048" layer="16"/>
+<wire x1="90.08" y1="40.73" x2="92.72" y2="43.37" width="0.3048" layer="16"/>
+<wire x1="92.72" y1="43.37" x2="92.72" y2="44.86" width="0.3048" layer="16"/>
+<wire x1="92.72" y1="44.86" x2="89.55" y2="44.86" width="0.3048" layer="16"/>
+<wire x1="89.55" y1="44.86" x2="87.4" y2="47.01" width="0.3048" layer="16"/>
+<wire x1="87.4" y1="47.01" x2="87.4" y2="53.28" width="0.3048" layer="16"/>
+<wire x1="87.4" y1="53.28" x2="87.41" y2="53.29" width="0.3048" layer="16"/>
+<wire x1="87.41" y1="53.29" x2="87.41" y2="53.61" width="0.3048" layer="16"/>
+<wire x1="87.41" y1="53.61" x2="87.39" y2="53.63" width="0.3048" layer="16"/>
+<via x="87.39" y="53.63" extent="1-16" drill="0.35"/>
+<wire x1="87.39" y1="53.63" x2="87.39" y2="58.81" width="0.3048" layer="1"/>
+<wire x1="88.4572" y1="59.8772" x2="88.4572" y2="60.6" width="0.3048" layer="1"/>
+<wire x1="87.39" y1="58.81" x2="88.4572" y2="59.8772" width="0.3048" layer="1"/>
+<wire x1="97.42" y1="31.9" x2="90.08" y2="39.24" width="0.3048" layer="16"/>
+<wire x1="88.4" y1="60.6" x2="88.4572" y2="60.6" width="0" layer="19" extent="1-1"/>
+</signal>
 </signals>
